Commit message: AIRoA試作機 納品バージョン

File: model/noid_lifter_mover.urdf.xacro (robot description, xacro)
@@ -5,8 +5,8 @@
     <xacro:include filename="$(arg parts_dir)/typeg_lifter/typeg_lifter.xacro" />
     <xacro:include filename="$(arg parts_dir)/typeg_mover/typeg_mover.xacro" />
-    <xacro:include filename="$(arg parts_dir)/trx_s/trx_s.xacro" />
     <xacro:include filename="$(arg parts_dir)/typeg_body/typeg_body.xacro" />
     <xacro:include filename="$(arg parts_dir)/typeg_larm/typeg_larm.xacro" />
     <xacro:include filename="$(arg parts_dir)/typeg_rarm/typeg_rarm.xacro" />
+    <xacro:include filename="$(arg parts_dir)/airoa_hand/airoa_hand.xacro" />
     <xacro:property name="robot_root" value="base_link" />
     <xacro:property name="lifter_bottom_link" value="lifter_bottom_link" />
@@ -15,8 +15,8 @@
     <xacro:property name="upper_base_link" value="waist_link" />
     <xacro:property name="larm_base_link" value="l_arm_link" />
-    <xacro:property name="larm_tip_link" value="l_wrist_r_link" />
+    <xacro:property name="larm_tip_link" value="l_wrist_p_link" />
     <xacro:property name="lhand_base_link" value="l_hand_link" />
     <xacro:property name="rarm_base_link" value="r_arm_link" />
-    <xacro:property name="rarm_tip_link" value="r_wrist_r_link" />
+    <xacro:property name="rarm_tip_link" value="r_wrist_p_link" />
     <xacro:property name="rhand_base_link" value="r_hand_link" />
     <xacro:typeg-mover
@@ -54,7 +54,7 @@
         <parent link="${rarm_tip_link}" />
         <child link="${rhand_base_link}" />
-        <origin xyz="0 0 -0.004" rpy="0 0 0 " />
+        <origin xyz="0 0 -0.0435" rpy="0 0 0 " />
     </joint>
-    <xacro:trx_s prefix="r" type="right" base_link="${rhand_base_link}"/>
+    <xacro:airoa_hand prefix="r" base_link="${rhand_base_link}"/>
     <xacro:typeg-larm base_link="${larm_base_link}" tip_link="${larm_tip_link}"/>
     <joint name="body_to_larm_connector" type="fixed">
@@ -66,7 +66,7 @@
         <parent link="${larm_tip_link}" />
         <child link="${lhand_base_link}" />
-        <origin xyz="0 0 -0.004" rpy="0 0 0 " />
+        <origin xyz="0 0 -0.0435" rpy="0 0 0 " />
     </joint>
-    <xacro:trx_s prefix="l" type="left" base_link="${lhand_base_link}"/>
+    <xacro:airoa_hand prefix="l" base_link="${lhand_base_link}"/>
     <xacro:include filename="$(find noid_lifter_mover)/model/noid_lifter_mover.ros2_control.xacro" />
     <xacro:noid_lifter_mover_ros2_control name="noid_lifter_mover" driver_settings="$(arg driver_settings)" />

File: model/parts/typeg_body/typeg_body.xacro (robot description, xacro)
@@ -4,10 +4,5 @@
     <xacro:include filename="$(arg parts_dir)/xacro_common.xacro" />
     <xacro:macro name="typeg-body" params="base_link">
-      <xacro:armlink
-         model_type="typeg_body"
-         link_name="${base_link}"
-         mesh_name="waist_link"
-         base_origin_xyz="0 0 0"
-         base_origin_rpy="0 0 0" />
+      <link name="${base_link}" />
       <xacro:armjoint
          joint_name="waist_y_joint"
@@ -16,5 +11,5 @@
          child="hip_sphere_link"
          joint_axis_xyz="0 0 1"
-         joint_origin_xyz="0 0 0.005"
+         joint_origin_xyz="0 0 0"
          joint_origin_rpy="0 0 0"
          joint_lower_limit="-2.09"
@@ -34,12 +29,11 @@
          child="hip_center"
          joint_axis_xyz="0 1 0"
-         joint_origin_xyz="0 0 0.132"
+         joint_origin_xyz="0 0 0.0655"
          joint_origin_rpy="0 0 0"
          joint_lower_limit="0.0"
-         joint_upper_limit="0.43"
+         joint_upper_limit="0.66"
          joint_velocity_limit="0.4"
          joint_effort_limit="10" />
-      <link name="hip_center">
-      </link>
+      <link name="hip_center" />
       <xacro:armjoint
          joint_name="waist_r_joint"
@@ -126,4 +120,12 @@
             <origin xyz="0 -0.055 0" rpy="0 0 0" />  <!-- realsense d415 -->
         </joint>
+      <xacro:armjoint
+            joint_name="head_camera_position"
+            type="fixed"
+            parent="head_link"
+            child="head_camera_link"
+            joint_origin_xyz="0.1516 0 0"
+            joint_origin_rpy="0 0 0" />
+        <link name="head_camera_link" />
     </xacro:macro>
 </root>

File: model/parts/typeg_larm/typeg_larm.xacro (robot description, xacro)
@@ -6,6 +6,5 @@
       name="typeg-larm"
       params="base_link tip_link">
-      <link name="${base_link}">
-      </link>
+      <link name="${base_link}" />
       <xacro:armjoint
          joint_name="l_shoulder_p_joint"
@@ -18,5 +17,5 @@
          joint_lower_limit="-1.48"
          joint_upper_limit="0.29"
-         joint_velocity_limit="0.4"
+         joint_velocity_limit="0.8"
          joint_effort_limit="10" />
       <xacro:armlink
@@ -36,5 +35,5 @@
          joint_lower_limit="-0.08"
          joint_upper_limit="1.57"
-         joint_velocity_limit="0.5"
+         joint_velocity_limit="1.0"
          joint_effort_limit="10" />
       <xacro:armlink
@@ -54,5 +53,5 @@
          joint_lower_limit="-1.57"
          joint_upper_limit="1.57"
-         joint_velocity_limit="1.1"
+         joint_velocity_limit="2.2"
          joint_effort_limit="10" />
       <xacro:armlink
@@ -68,9 +67,9 @@
          child="l_elbow_virtual_link"
          joint_axis_xyz="0 1 0"
-         joint_origin_xyz="0.0 0 -0.2085"
+         joint_origin_xyz="0.0 0 -0.2385"
          joint_origin_rpy="0 0 0"
          joint_lower_limit="-3.0"
          joint_upper_limit="0"
-         joint_velocity_limit="1.1"
+         joint_velocity_limit="2.2"
          joint_effort_limit="10" />
       <link name="l_elbow_virtual_link">
@@ -136,5 +135,5 @@
          joint_lower_limit="-1.57"
          joint_upper_limit="1.57"
-         joint_velocity_limit="1.2"
+         joint_velocity_limit="2.4"
          joint_effort_limit="10" />
       <xacro:armlink
@@ -145,37 +144,37 @@
          base_origin_rpy="0 0 0" />
       <xacro:armjoint
-         joint_name="l_wrist_p_joint"
+         joint_name="l_wrist_r_joint"
          type="revolute"
          parent="l_forearm_link"
-         child="l_wrist_center"
-         joint_axis_xyz="0 1 0"
+         child="l_wrist_r_link"
+         joint_axis_xyz="1 0 0"
          joint_origin_xyz="0 0 -0.124"
          joint_origin_rpy="0 0 0"
-         joint_lower_limit="-0.08"
-         joint_upper_limit="0.08"
-         joint_velocity_limit="0.8"
+         joint_lower_limit="-0.73"
+         joint_upper_limit="0.52"
+         joint_velocity_limit="3.6"
          joint_effort_limit="10" />
       <xacro:armlink
          model_type="typeg_larm"
-         link_name="l_wrist_center"
-         mesh_name="l_wrist_center_link"
+         link_name="l_wrist_r_link"
+         mesh_name="l_wrist_r_link"
          base_origin_xyz="0 0 0"
          base_origin_rpy="0 0 0" />
       <xacro:armjoint
-         joint_name="l_wrist_r_joint"
+         joint_name="l_wrist_p_joint"
          type="revolute"
-         parent="l_wrist_center"
-         child="l_wrist_r_link"
-         joint_axis_xyz="1 0 0"
+         parent="l_wrist_r_link"
+         child="l_wrist_p_link"
+         joint_axis_xyz="0 1 0"
          joint_origin_xyz="0 0 0"
          joint_origin_rpy="0 0 0"
          joint_lower_limit="-1.57"
-         joint_upper_limit="0.0"
-         joint_velocity_limit="1.8"
+         joint_upper_limit="1.57"
+         joint_velocity_limit="3.6"
          joint_effort_limit="10" />
       <xacro:armlink
          model_type="typeg_larm"
          link_name="${tip_link}"
-         mesh_name="l_wrist_r_link"
+         mesh_name="l_wrist_p_link"
          base_origin_xyz="0 0 0"
          base_origin_rpy="0 0 0" />

File: model/parts/typeg_lifter/typeg_lifter.xacro (robot description, xacro)
@@ -18,5 +18,5 @@
          child="leg_shank_link_dummy"
          joint_axis_xyz="0 -1 0"
-         joint_origin_xyz="0.01982 0 0.06182"
+         joint_origin_xyz="0.01982 0 0.06682"
          joint_origin_rpy="0 0 0"
          mimic_parent="ankle_joint"
@@ -36,5 +36,5 @@
          child="leg_shank_link"
          joint_axis_xyz="0 -1 0"
-         joint_origin_xyz="-0.012 0 0.03"
+         joint_origin_xyz="-0.012 0 0.035"
          joint_origin_rpy="0 0 0"
          joint_lower_limit="0"
@@ -54,5 +54,5 @@
          child="leg_knee_link"
          joint_axis_xyz="0 -1 0"
-         joint_origin_xyz="0 0 0.25"
+         joint_origin_xyz="0 0 0.37"
          joint_origin_rpy="0 0 0"
          mimic_parent="ankle_joint"
@@ -108,5 +108,5 @@
          child="leg_base_link"
          joint_axis_xyz="0 -1 0"
-         joint_origin_xyz="0 0 0.25"
+         joint_origin_xyz="0 0 0.37"
          joint_origin_rpy="0 0 0"
          mimic_parent="knee_joint"
@@ -126,5 +126,5 @@
          child="${top_link}"
          joint_axis_xyz="0 0 1"
-         joint_origin_xyz="0.012 0 0.040"
+         joint_origin_xyz="0.012 0 0.085"
          joint_origin_rpy="0 0 0" />
       <link name="${top_link}" />

File: model/parts/typeg_mover/typeg_mover.xacro (robot description, xacro)
@@ -23,18 +23,12 @@
          base_origin_xyz="0 0 0"
          base_origin_rpy="0 0 0" />
+      <link name="${top_link}" />
       <xacro:armjoint
          joint_name="wheels_body_to_top_connector"
          type="fixed"
-         parent="wheel_base_link"
+         parent="${base_link}"
          child="${top_link}"
-         joint_origin_xyz="0.0 0.0 0.087"
+         joint_origin_xyz="0.026 0.0 0.237"
          joint_origin_rpy="0 0 0" />
-      <xacro:armlink
-         model_type="typeg_mover"
-         link_name="${top_link}"
-         mesh_name="wheels_top"
-         base_origin_xyz="0 0 0"
-         base_origin_rpy="0 0 0" />
-      <!-- ホイール -->
       <xacro:armjoint
          joint_name="wheels_body_to_front_left_mecanum_connector"
@@ -48,7 +42,7 @@
          model_type="typeg_mover"
          link_name="wheels_front_left_mecanum"
-         mesh_name="wheels_mecanum"
+         mesh_name="wheels_mecanum_B"
          base_origin_xyz="0 0 0"
-         base_origin_rpy="${-pi/2} 0 0" />
+         base_origin_rpy="0 0 0" />
       <xacro:armjoint
          joint_name="wheels_body_to_front_right_mecanum_connector"
@@ -62,7 +56,7 @@
          model_type="typeg_mover"
          link_name="wheels_front_right_mecanum"
-         mesh_name="wheels_mecanum"
+         mesh_name="wheels_mecanum_A"
          base_origin_xyz="0 0 0"
-         base_origin_rpy="${-pi/2} 0 0" />
+         base_origin_rpy="0 0 0" />
       <xacro:armjoint
          joint_name="wheels_body_to_rear_left_mecanum_connector"
@@ -76,7 +70,7 @@
          model_type="typeg_mover"
          link_name="wheels_rear_left_mecanum"
-         mesh_name="wheels_mecanum"
+         mesh_name="wheels_mecanum_A"
          base_origin_xyz="0 0 0"
-         base_origin_rpy="${-pi/2} 0 0" />
+         base_origin_rpy="0 0 0" />
       <xacro:armjoint
          joint_name="wheels_body_to_rear_right_mecanum_connector"
@@ -90,8 +84,7 @@
          model_type="typeg_mover"
          link_name="wheels_rear_right_mecanum"
-         mesh_name="wheels_mecanum"
+         mesh_name="wheels_mecanum_B"
          base_origin_xyz="0 0 0"
-         base_origin_rpy="${-pi/2} 0 0" />
-      <!-- LIDAR -->
+         base_origin_rpy="0 0 0" />
       <xacro:armjoint
          joint_name="wheels_body_to_base_laser_connector"
@@ -99,5 +92,5 @@
          parent="wheel_base_link"
          child="wheels_base_laser_link"
-         joint_origin_xyz="0.308 0 0.1014"
+         joint_origin_xyz="0.296 0 0.1014"
          joint_origin_rpy="0 0 0" />
       <xacro:armlink
@@ -107,53 +100,4 @@
          base_origin_xyz="0 0 0"
          base_origin_rpy="0 0 0" />
-      <!-- カメラ -->
-      <xacro:armjoint
-         joint_name="wheel_base_link_to_front_camera_base_link"
-         type="fixed"
-         parent="wheel_base_link"
-         child="front_camera_base_link"
-         joint_origin_xyz="0.31815 0 0.0185"
-         joint_origin_rpy="0 0 0" />
-      <link name="front_camera_base_link" />
-      <xacro:armjoint
-         joint_name="front_camera_base_link_to_front_camera_link"
-         type="fixed"
-         parent="front_camera_base_link"
-         child="front_camera_link"
-         joint_origin_xyz="0 0.0175 0.0125"
-         joint_origin_rpy="0 0 0" />
-      <link name="front_camera_link" />
-      <xacro:armjoint
-         joint_name="front_camera_link_to_front_camera_right_ir_link"
-         type="fixed"
-         parent="front_camera_link"
-         child="front_camera_right_ir_frame"
-         joint_origin_xyz="0 -0.05 0"
-         joint_origin_rpy="0 0 0" />
-      <link name="front_camera_right_ir_frame" />
-      <xacro:armjoint
-         joint_name="wheel_base_link_to_rear_camera_base_link"
-         type="fixed"
-         parent="wheel_base_link"
-         child="rear_camera_base_link"
-         joint_origin_xyz="-0.31815 0 0.0185"
-         joint_origin_rpy="0 0 ${pi}" />
-      <link name="rear_camera_base_link" />
-      <xacro:armjoint
-         joint_name="rear_camera_base_link_to_rear_camera_link"
-         type="fixed"
-         parent="rear_camera_base_link"
-         child="rear_camera_link"
-         joint_origin_xyz="0 0.0175 0.0125"
-         joint_origin_rpy="0 0 0" />
-      <link name="rear_camera_link" />
-      <xacro:armjoint
-         joint_name="rear_camera_link_to_rear_camera_right_ir_link"
-         type="fixed"
-         parent="rear_camera_link"
-         child="rear_camera_right_ir_frame"
-         joint_origin_xyz="0 -0.05 0"
-         joint_origin_rpy="0 0 0" />
-      <link name="rear_camera_right_ir_frame" />
    </xacro:macro>
 </root>

File: model/parts/typeg_rarm/typeg_rarm.xacro (robot description, xacro)
@@ -6,6 +6,5 @@
       name="typeg-rarm"
       params="base_link tip_link">
-      <link name="${base_link}">
-      </link>
+      <link name="${base_link}" />
       <xacro:armjoint
          joint_name="r_shoulder_p_joint"
@@ -18,5 +17,5 @@
          joint_lower_limit="-1.48"
          joint_upper_limit="0.29"
-         joint_velocity_limit="0.4"
+         joint_velocity_limit="0.8"
          joint_effort_limit="10" />
       <xacro:armlink
@@ -36,5 +35,5 @@
          joint_lower_limit="-1.57"
          joint_upper_limit="0.08"
-         joint_velocity_limit="0.5"
+         joint_velocity_limit="1.0"
          joint_effort_limit="10" />
       <xacro:armlink
@@ -54,5 +53,5 @@
          joint_lower_limit="-1.57"
          joint_upper_limit="1.57"
-         joint_velocity_limit="1.1"
+         joint_velocity_limit="2.2"
          joint_effort_limit="10" />
       <xacro:armlink
@@ -68,9 +67,9 @@
          child="r_elbow_virtual_link"
          joint_axis_xyz="0 1 0"
-         joint_origin_xyz="0.0 0 -0.2085"
+         joint_origin_xyz="0.0 0 -0.2385"
          joint_origin_rpy="0 0 0"
          joint_lower_limit="-3.0"
          joint_upper_limit="0"
-         joint_velocity_limit="1.1"
+         joint_velocity_limit="2.2"
          joint_effort_limit="10" />
       <link name="r_elbow_virtual_link">
@@ -136,5 +135,5 @@
          joint_lower_limit="-1.57"
          joint_upper_limit="1.57"
-         joint_velocity_limit="1.2"
+         joint_velocity_limit="2.4"
          joint_effort_limit="10" />
       <xacro:armlink
@@ -145,37 +144,37 @@
          base_origin_rpy="0 0 0" />
       <xacro:armjoint
-         joint_name="r_wrist_p_joint"
+         joint_name="r_wrist_r_joint"
          type="revolute"
          parent="r_forearm_link"
-         child="r_wrist_center"
-         joint_axis_xyz="0 1 0"
+         child="r_wrist_r_link"
+         joint_axis_xyz="1 0 0"
          joint_origin_xyz="0 0 -0.124"
          joint_origin_rpy="0 0 0"
-         joint_lower_limit="-0.08"
-         joint_upper_limit="0.08"
-         joint_velocity_limit="0.8"
+         joint_lower_limit="-0.52"
+         joint_upper_limit="0.73"
+         joint_velocity_limit="3.6"
          joint_effort_limit="10" />
       <xacro:armlink
          model_type="typeg_rarm"
-         link_name="r_wrist_center"
-         mesh_name="r_wrist_center_link"
+         link_name="r_wrist_r_link"
+         mesh_name="r_wrist_r_link"
          base_origin_xyz="0 0 0"
          base_origin_rpy="0 0 0" />
       <xacro:armjoint
-         joint_name="r_wrist_r_joint"
+         joint_name="r_wrist_p_joint"
          type="revolute"
-         parent="r_wrist_center"
-         child="r_wrist_r_link"
-         joint_axis_xyz="1 0 0"
+         parent="r_wrist_r_link"
+         child="r_wrist_p_link"
+         joint_axis_xyz="0 1 0"
          joint_origin_xyz="0 0 0"
          joint_origin_rpy="0 0 0"
-         joint_lower_limit="0.0"
+         joint_lower_limit="-1.57"
          joint_upper_limit="1.57"
-         joint_velocity_limit="1.8"
+         joint_velocity_limit="3.6"
          joint_effort_limit="10" />
       <xacro:armlink
          model_type="typeg_rarm"
          link_name="${tip_link}"
-         mesh_name="r_wrist_r_link"
+         mesh_name="r_wrist_p_link"
          base_origin_xyz="0 0 0"
          base_origin_rpy="0 0 0" />

File: model/parts/xacro_common.xacro (robot description, xacro)
@@ -26,5 +26,5 @@
             <child link="${child}" />
             <origin xyz="${joint_origin_xyz}" rpy="${joint_origin_rpy}" />
-            <xacro:unless value="${type=='fixed' or mimic}">
+            <xacro:unless value="${type=='fixed' or type=='continuous'}">
                 <limit effort="${joint_effort_limit}" velocity="${joint_velocity_limit}" lower="${joint_lower_limit}" upper="${joint_upper_limit}" />
             </xacro:unless>
